File: AL8843-esp32-led-board.kicad_pcb (KiCad board)
At the start: 2 copper layers, 36.1 x 26.8 mm, 16 parts, among them IC1 AL8843QSP-13

Commit message: jlcpcb order W2025081219518153
Parts:
- R1, R2: footprint Resistor_SMD:R_1206_3216Metric -> Resistor_SMD:R_2512_6332Metric
- moved R1 2.65 mm to (61.5, 27.8)
- moved REF** 1.95 mm to (55.2, 29.0)
- moved C4 1.80 mm to (70.0, 33.5)
- moved C5 1.80 mm to (68.5, 33.5)
- moved REF** 0.96 mm to (67.8, 29.0)
- moved R2 0.95 mm to (61.5, 31.8)
Connections:
- IC1 pad 4: LED_A_+ -> unconnected-(IC1-NC-Pad4)
Other:
- board size 36.1 x 26.8 mm -> 36.2 x 28.8 mm

Commit message: ESP32 power
Parts:
- added C10: 0.47uF 100V X7R 1206, Capacitor_SMD:C_1206_3216Metric, F.Cu at (49.2, 57.5)
- added C11: 0.47uF 100V X7R 1206, Capacitor_SMD:C_1206_3216Metric, F.Cu at (60.8, 74.0)
- added C12: 0.47uF 100V X7R 1206, Capacitor_SMD:C_1206_3216Metric, F.Cu at (72.9, 58.6)
- added C6: 0.022uF 100V X7R, Capacitor_SMD:C_0603_1608Metric, F.Cu at (47.2, 57.2)
- added C7: 0.22uF 16V X7R, Capacitor_SMD:C_0402_1005Metric, F.Cu at (71.2, 59.7)
- added C8: 100uF Polymer Hybrid 50V 28ohm 10x10SMD, Capacitor_SMD:C_Elec_10x10.2, F.Cu at (45.4, 49.8)
- added C9: 330uF AL 35V 0.06ohm, Capacitor_SMD:CP_Elec_8x10, F.Cu at (66.5, 72.5)
- added D2: D_Schottky, Diode_SMD:D_SMC, F.Cu at (55.8, 72.3)
- added IC2: LM2596SX-5.0_NOPB, LM2596SX-5.0:KTT0005B, F.Cu at (45.7, 74.5)
- added L2: 47uH 6.5A 0.076ohm AEC-Q200 Grade 0, Inductor_SMD:L_TechFuse_SL1265, F.Cu at (59.4, 60.5)
- added OFF: Pin_D1.0mm_L10.0mm, Connector_Pin:Pin_D1.0mm_L10.0mm, F.Cu at (72.4, 66.3)
- added R4: 1.02K 1% 0.25W, Resistor_SMD:R_1206_3216Metric, F.Cu at (72.6, 70.7)
- added REF**: ESP32_C3_Super_mini, ESP32-C3-super-mini:ESP32_C3_Super_mini, F.Cu at (74.2, 55.6)
- moved CTRL 22.6 mm to (68.1, 46.0)
- moved R3 18.3 mm to (68.1, 41.1), turned to 90 degrees
- moved REF** 15.0 mm to (89.0, 36.4)
Connections:
- IC1 pad 4: unconnected-(IC1-NC-Pad4) -> LED_A_+
Routing:
- net +5V: track 0.00 -> 60.6 mm
- net OFF: track 0.00 -> 37.5 mm, vias 0 -> 1
- net CTRL: track 3.24 -> 35.4 mm, vias 0 -> 1
- net Net-(D2-K): track 0.00 -> 21.7 mm
- net Net-(IC1-CTRL): track 10.8 -> 13.0 mm
- net GND: vias 15 -> 62
Other:
- board size 36.2 x 28.8 mm -> 55.5 x 54.8 mm

Commit message: misc
Parts:
- removed the REF** at (74.2, 55.6)
- added GND: Pin_D1.0mm_L10.0mm, Connector_Pin:Pin_D1.0mm_L10.0mm, F.Cu at (48.8, 41.5)
- added GND: Pin_D1.0mm_L10.0mm, Connector_Pin:Pin_D1.0mm_L10.0mm, F.Cu at (71.0, 55.8)
- added REF**: XIAO-ESP32-C3-DIP, Seeed Studio XIAO Series Library:XIAO-ESP32C3-DIP, F.Cu at (84.5, 67.8)
- moved C7 15.6 mm to (71.5, 75.3), turned to 90 degrees
- moved C12 15.6 mm to (73.2, 74.2), turned to 90 degrees
- moved R4 8.30 mm to (71.0, 62.5), turned to -90 degrees
- moved OFF 1.47 mm to (71.1, 67.0)
Routing:
- net CTRL: track 35.4 -> 3.42 mm, vias 1 -> 0
- net +5V: track 60.6 -> 52.9 mm
- net Net-(D2-K): track 21.7 -> 17.6 mm
- net OFF: track 37.5 -> 36.5 mm
- net GND: track 0.00 -> 0.16 mm, vias 62 -> 63
Other:
- board size 55.5 x 54.8 mm -> 59 x 54.8 mm
